File: hardware/pcb/stm32_esp32_pcb/stm32_esp32_pcb.kicad_sch (KiCad schematic)
At the start: 45 parts, among them J1 Conn_01x06_STM32, J2 Conn_01x06_Pin, Q1 TEPT4400, SW1 SW_Push, U1 STM32L031F6Px, U2 LM2904, U3 XC6220B331MR, U4 ESP32-WROOM-32U, U5 LP2985-3.3, Y1 Crystal

Commit message: update
Parts:
- removed J1: Conn_01x06_STM32, SNES:PinHeader_1x06_P2.54mm_Vertical_STM32, symbol SNES:Conn_01x06_STM32
- added J1: Conn_01x06_Pin, Connector_PinHeader_2.54mm:PinHeader_1x06_P2.54mm_Horizontal, symbol Connector:Conn_01x06_Pin
- added J3: Conn_01x02_Pin, symbol Connector:Conn_01x02_Pin
- added MOD1: TP4056 MODULE, TP4056-Module:TP4056-Module, symbol SNES:TP4056_MODULE
- added R16, R17: R0603_100k_1%_100mW_100PPM_AC, Resistor_SMD:R_0603_1608Metric, symbol Resistors_SMD_0603:R0603_100k_1%_100mW_100PPM_AC
Connections:
- net +3V3: now also J1.1 (Pin_1), J3.1 (Pin_1); no longer Q1.1 (C)
- net GND: now also J1.3 (Pin_3), MOD1.4 (OUT-), R17.2; no longer BT1.1-, BT1.2-
- net NRST: now also J1.5 (Pin_5)
- net SWCLK: now also J1.2 (Pin_2)
- net SWDIO: now also J1.4 (Pin_4)
- net SWO: now also J1.6 (Pin_6)
- net VBUS: now also MOD1.3 (OUT+), R16.1
- net V_SENS: now also R16.2, R17.1
- net EMITER: now reaches C16.1, R15.1
- net EMITER: now also J3.2 (Pin_2); no longer Q1.2 (E)
- net +BATT renamed B+
- net B+: now also MOD1.5 (B+)
- new net B-: BT1.1-, BT1.2-, MOD1.6 (B-)
Other:
- title: (none) -> WIFI meter pulse counter
- moved on the sheet: BT1, C16, Q1, R10, R11, R12, R13, R14, R15, R8, R9, RV1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

Commit message: Update
Parts:
- removed Q1: TEPT4400, LED_THT:LED_D3.0mm_Clear, symbol Sensor_Optical:TEPT4400
- added C17, C18: C0603_100nF_16V_X7R, Capacitor_SMD:C_0603_1608Metric, symbol Capacitors_SMD_0603:C0603_100nF_16V_X7R
Connections:
- net +3V3: now also C18.2
- net GND: now also C17.2, C18.1
- net V_SENS: now also C17.1
Other:
- note added: "TEPT4400"
- moved on the sheet: C1, C2, R16, R17, R9, Y1

Commit message: DRX check
54 DRC errors left
Parts:
- removed R1, R2, R3, R4, R5: R0402_10k_1%_62.5mW_100PPM_AC, Resistor_SMD:R_0402_1005Metric, symbol Resistors_SMD_0402:R0402_10k_1%_62.5mW_100PPM_AC
- added R1, R2, R3, R4, R5: R0603_10k_1%_100mW_100PPM_AC, Resistor_SMD:R_0603_1608Metric, symbol Resistors_SMD_0603:R0603_10k_1%_100mW_100PPM_AC
Connections:
- net +3V3: now also R2.1, R3.1; no longer J2.1 (Pin_1)
- net BOOT0: now also R4.1
- net EN: now also R5.2
- net ESP32_E: now also R2.2
- net GND: now also R4.2
- net IO00: now also R1.2
- net NRST: now also R3.2
- net +3V3_ESP renamed +3.3VDAC
- net +3.3VDAC: now also J2.1 (Pin_1), R1.1, R5.1

Commit message: update
Almos done
Parts:
- Y1: footprint Crystal:Crystal_AT310_D3.0mm_L10.0mm_Horizontal -> Crystal:Crystal_C38-LF_D3.0mm_L8.0mm_Horizontal_1EP_style1
Changed lines of the file:
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@@
       (effects (font (size 1.27 1.27)) (justify right))
     )
-    (property "Footprint" "Crystal:Crystal_AT310_D3.0mm_L10.0mm_Horizontal" (at 31.75 71.12 0)
+    (property "Footprint" "Crystal:Crystal_C38-LF_D3.0mm_L8.0mm_Horizontal_1EP_style1" (at 31.75 71.12 0)
       (effects (font (size 1.27 1.27)) hide)
     )

Commit message: Update
Parts:
- removed D1, D2: 1N4148W, Diode_SMD:D_SOD-123, symbol Diode:1N4148W
- removed SW1: SW_Push, Button_Switch_THT:SW_PUSH_6mm_H4.3mm, symbol Switch:SW_Push
- added D1, D2: BAT54C, Package_TO_SOT_SMD:SOT-23, symbol Diode:BAT54C
- added J4, J5: Conn_01x02_Pin, Connector_PinHeader_2.54mm:PinHeader_1x02_P2.54mm_Vertical, symbol Connector:Conn_01x02_Pin
- J3: footprint (none) -> Connector_PinHeader_2.54mm:PinHeader_1x02_P2.54mm_Horizontal
Connections:
- net +3V3: now also J3.2 (Pin_2); no longer J3.1 (Pin_1)
- net BOOT0: now also D2.1
- net EMITER: now also J3.1 (Pin_1); no longer J3.2 (Pin_2)
- net EN: now also D2.2
- net GND: now also J4.2 (Pin_2), J5.2 (Pin_2)
- net IO00: now also D1.2
- net NRST: now also D1.1
- new net ESP32: D1.3, J4.1 (Pin_1)
- new net STM32: D2.3, J5.1 (Pin_1)
