File: hardware/pcb/stm32_esp32_pcb/stm32_esp32_pcb.kicad_pcb (KiCad board)
At the start: 2 copper layers, 88 x 60 mm, 45 parts, among them J1 Conn_01x06_STM32, J2 Conn_01x06_Pin, Q1 TEPT4400, SW1 SW_Push, U1 STM32L031F6Px, U2 LM2904, U3 XC6220B331MR, U4 ESP32-WROOM-32U, U5 LP2985-3.3, Y1 Crystal

Commit message: update
Parts:
- added MOD1: TP4056 MODULE, TP4056-Module:TP4056-Module, F.Cu at (151.6, 89.5)
- added R16: R0603_100k_1%_100mW_100PPM_AC, Resistor_SMD:R_0603_1608Metric, F.Cu at (166.2, 66.0)
- added R17: R0603_100k_1%_100mW_100PPM_AC, Resistor_SMD:R_0603_1608Metric, F.Cu at (166.2, 68.5)
- J1: value Conn_01x06_STM32 -> Conn_01x06_Pin; footprint SNES:PinHeader_1x06_P2.54mm_Vertical_STM32 -> Connector_PinHeader_2.54mm:PinHeader_1x06_P2.54mm_Horizontal
- moved C10 105.5 mm to (192.6, 86.8), turned to -90 degrees
- moved C9 101.8 mm to (190.8, 87.0), turned to -90 degrees
- moved C12 101.3 mm to (204.3, 84.9), turned to 90 degrees
- moved C14 95.3 mm to (202.5, 85.0), turned to 90 degrees
- moved C13 93.4 mm to (196.3, 84.9), turned to 90 degrees
- moved C15 87.2 mm to (194.4, 85.1), turned to 90 degrees
- moved U5 54.1 mm to (154.5, 69.0)
- moved J2 44.3 mm to (179.0, 59.5), turned to 90 degrees
- moved SW1 44.2 mm to (204.2, 39.2)
- moved U3 38.8 mm to (199.6, 84.9), turned to 180 degrees
- moved J1 34.0 mm to (158.7, 59.5), turned to 90 degrees
- moved U2 28.7 mm to (197.5, 68.0), turned to 180 degrees
- moved U4 18.8 mm to (179.9, 79.4), turned to 180 degrees
- moved U1 11.9 mm to (160.5, 80.0)
Connections:
- net +BATT renamed /B+
- BT1 pad 1-: GND -> /B-
- BT1 pad 2-: GND -> /B-
- C16 pad 1: Net-(Q1-E) -> /EMITER
- Q1 pad 1: +3V3 -> unconnected-(Q1-C-Pad1)
- Q1 pad 2: Net-(Q1-E) -> unconnected-(Q1-E-Pad2)
- R15 pad 1: Net-(Q1-E) -> /EMITER
Routing:
- net /+3V3_ESP: track 0.00 -> 10.0 mm
- net GND: track 0.00 -> 6.71 mm, vias 0 -> 2
- added copper zone on In2.Cu, net /B+
- added copper zone on In2.Cu, net /B-
- added copper zone on In1.Cu, net GND
- added copper zone on In2.Cu, net VBUS
Other:
- board size 88 x 60 mm -> 78.2 x 40.8 mm
- copper layers 2 -> 4
- rule pad_to_mask_clearance: 0 -> 0.051
- board text added: "3V3"
- board text added: "EN"
- board text added: "GND"
- board text added: "IO0"
- board text added: "NRST"
- board text added: "RX"
- board text added: "SWCLK"
- board text added: "SWDIO"
- board text added: "SWO"
- board text added: "TX"
- board text added: "v${Revision}"

Commit message: Update
Parts:
- removed Q1: TEPT4400, LED_THT:LED_D3.0mm_Clear
- added C17: C0603_100nF_16V_X7R, Capacitor_SMD:C_0603_1608Metric, F.Cu at (116.2, 74.5)
- added C18: C0603_100nF_16V_X7R, Capacitor_SMD:C_0603_1608Metric, F.Cu at (116.2, 77.0)
- moved R2 105.0 mm to (200.0, 82.5)
- moved R12 91.4 mm to (204.0, 67.0), turned to 90 degrees
- moved R11 91.3 mm to (204.0, 70.0), turned to -90 degrees
- moved R1 89.6 mm to (188.5, 64.2)
- moved R9 86.1 mm to (198.8, 65.0), turned to 180 degrees
- moved R8 82.1 mm to (194.5, 67.2), turned to -90 degrees
- moved R13 81.9 mm to (194.5, 70.2), turned to -90 degrees
- moved R14 80.5 mm to (193.0, 70.2), turned to 90 degrees
- moved R10 80.3 mm to (193.0, 67.2), turned to 90 degrees
- moved C7 65.5 mm to (161.0, 66.8)
- moved C3 65.4 mm to (158.0, 71.0), turned to -90 degrees
- moved C8 65.3 mm to (161.0, 68.2)
- moved C5 62.2 mm to (155.5, 71.0), turned to -90 degrees
- moved C4 50.4 mm to (152.8, 65.8), turned to 90 degrees
- moved R17 14.2 mm to (152.8, 73.0), turned to -90 degrees
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Routing:
- added copper zone on In2.Cu, net +3V3

Commit message: update
Parts:
- moved C11 85.4 mm to (196.8, 72.8), turned to -90 degrees
- moved C6 69.3 mm to (155.5, 80.4), turned to -90 degrees
- moved C18 49.1 mm to (165.2, 80.7), turned to 90 degrees
- moved R2 1.14 mm to (199.1, 81.8), turned to -90 degrees
- moved MOD1 0.58 mm to (151.6, 89.5)
Routing:
- net /RX: track 0.00 -> 62.9 mm, vias 0 -> 1
- net /PULSE: track 0.00 -> 60.9 mm, vias 0 -> 2
- net /TX: track 0.00 -> 52.9 mm, vias 0 -> 1
- net /ESP32_E: track 0.00 -> 48.4 mm, vias 0 -> 3
- net /NRST: track 0.00 -> 36.4 mm, vias 0 -> 2
- net /EN: track 0.00 -> 27.6 mm
- net /SWCLK: track 0.00 -> 26.1 mm
- net GND: track 6.71 -> 31.8 mm, vias 2 -> 19
- net /SWDIO: track 0.00 -> 23.2 mm
- net /BOOT0: track 0.00 -> 17.8 mm, vias 0 -> 2
- net /V_SENS: track 0.00 -> 16.6 mm
- net VBUS: track 0.00 -> 16.2 mm, vias 0 -> 3
- net +3V3: track 0.00 -> 15.0 mm, vias 0 -> 6
- net /SCL: track 0.00 -> 12.4 mm, vias 0 -> 2
- net /SDA: track 0.00 -> 9.01 mm
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
Commit message: DRX check
54 DRC errors left
Parts:
- R1, R2, R3, R4, R5: value R0402_10k_1%_62.5mW_100PPM_AC -> R0603_10k_1%_100mW_100PPM_AC; footprint Resistor_SMD:R_0402_1005Metric -> Resistor_SMD:R_0603_1608Metric
- moved R5 93.3 mm to (191.4, 76.2), turned to 180 degrees
- moved R4 70.4 mm to (169.6, 66.9), turned to 90 degrees
- moved R3 67.1 mm to (164.6, 71.0)
- moved R1 4.37 mm to (192.5, 62.5), turned to 180 degrees
- moved R2 0.85 mm to (199.7, 81.2)
- moved C6 0.27 mm to (155.5, 80.7)
Connections:
- C10 pad 1: /+3V3_ESP -> +3.3VDAC
- C13 pad 1: /+3V3_ESP -> +3.3VDAC
- C15 pad 1: /+3V3_ESP -> +3.3VDAC
- C9 pad 1: /+3V3_ESP -> +3.3VDAC
- J2 pad 1: +3V3 -> +3.3VDAC
- R1 pad 1: /+3V3_ESP -> +3.3VDAC
- R1 pad 2: /EN -> /IO00
- R5 pad 1: /+3V3_ESP -> +3.3VDAC
- R5 pad 2: /IO00 -> /EN
- R6 pad 1: /+3V3_ESP -> +3.3VDAC
- R7 pad 1: /+3V3_ESP -> +3.3VDAC
- U3 pad 5: /+3V3_ESP -> +3.3VDAC
- U4 pad 2: /+3V3_ESP -> +3.3VDAC
Routing:
- net +3.3VDAC: track 0.00 -> 58.0 mm, vias 0 -> 3
- net /+3V3_ESP: track 10.0 -> 0.00 mm
- net /BOOT0: track 17.8 -> 22.6 mm
- net GND: track 31.8 -> 34.3 mm, vias 19 -> 22
- net +3V3: track 15.0 -> 14.2 mm
- net /ESP32_E: vias 3 -> 2

Commit message: update
Almos done
Parts:
- Y1: footprint Crystal:Crystal_AT310_D3.0mm_L10.0mm_Horizontal -> Crystal:Crystal_C38-LF_D3.0mm_L8.0mm_Horizontal_1EP_style1
- moved R6 194.6 mm to (192.4, 80.2), turned to 180 degrees
- moved R7 194.4 mm to (192.4, 81.8), turned to 180 degrees
- moved Y1 60.3 mm to (153.8, 78.0)
- moved C16 54.2 mm to (205.5, 67.0), turned to -90 degrees
- moved R15 52.0 mm to (205.5, 64.0), turned to 90 degrees
- moved C2 50.7 mm to (155.8, 75.7), turned to -90 degrees
- moved C1 49.4 mm to (153.8, 75.7), turned to -90 degrees
- moved C17 47.1 mm to (163.3, 75.4)
- moved R3 7.46 mm to (170.1, 65.9), turned to 180 degrees
- moved C18 3.01 mm to (168.2, 80.4)
- moved C6 3.01 mm to (158.5, 80.4)
- moved U1 3.01 mm to (163.5, 79.7)
- moved R4 2.39 mm to (171.8, 67.7), turned to 0 degrees
- moved R1 2.38 mm to (193.1, 64.8)
- moved R17 0.95 mm to (152.7, 72.0)
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Routing:
- net /SCL: track 12.4 -> 42.1 mm, vias 2 -> 3
- net /IO00: track 0.00 -> 24.6 mm, vias 0 -> 2
- net /SDA: track 9.01 -> 32.4 mm, vias 0 -> 2
- net /OSC2: track 0.00 -> 9.16 mm
- net /NRST: track 36.4 -> 29.1 mm
- net /PULSE: track 60.9 -> 53.7 mm
- net /OSC1: track 0.00 -> 6.70 mm
- net /RX: track 62.9 -> 56.8 mm
- net /TX: track 52.9 -> 47.9 mm
- net /SWCLK: track 26.1 -> 22.6 mm
- net /BOOT0: track 22.6 -> 19.2 mm
- net GND: track 34.3 -> 37.4 mm, vias 22 -> 25
- net /SWDIO: track 23.2 -> 20.2 mm
- net /ESP32_E: track 48.4 -> 50.9 mm
- net /V_SENS: track 16.6 -> 19.1 mm
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Other:
- rule solder_mask_min_width: 0.25 -> 0.1
- board text added: "JKBI"

Commit message: DRC check
11 DRC errors left
Parts:
- moved RV1 71.6 mm to (200.2, 59.5), turned to 90 degrees
- moved R9 1.98 mm to (196.9, 64.3), turned to -90 degrees
Routing:
- net Net-(U2A--): track 2.29 -> 14.8 mm
- net Net-(R9-Pad1): track 7.13 -> 14.1 mm
- net /IO00: track 24.6 -> 29.3 mm
- net GND: track 37.4 -> 39.0 mm, vias 25 -> 27
- net Net-(U2B-+): track 4.81 -> 4.14 mm

Commit message: Update
Parts:
- removed SW1: SW_Push, Button_Switch_THT:SW_PUSH_6mm_H4.3mm
- added J3: Conn_01x02_Pin, Connector_PinHeader_2.54mm:PinHeader_1x02_P2.54mm_Horizontal, F.Cu at (199.3, 73.5)
- added J4: Conn_01x02_Pin, Connector_PinHeader_2.54mm:PinHeader_1x02_P2.54mm_Vertical, F.Cu at (175.2, 59.5)
- added J5: Conn_01x02_Pin, Connector_PinHeader_2.54mm:PinHeader_1x02_P2.54mm_Vertical, F.Cu at (155.1, 59.5)
- D1, D2: value 1N4148W -> BAT54C; footprint Diode_SMD:D_SOD-123 -> Package_TO_SOT_SMD:SOT-23
- moved D1 47.4 mm to (175.2, 63.4), turned to 90 degrees
- moved D2 35.1 mm to (156.2, 63.0), turned to 180 degrees
- moved R4 7.05 mm to (164.8, 67.8), turned to -90 degrees
- moved R3 0.81 mm to (170.6, 65.3), turned to 90 degrees
- moved RV1 0.76 mm to (200.9, 59.2)
Connections:
- D1 pad 2: Net-(D1-A) -> /IO00
- D2 pad 1: /IO00 -> /BOOT0
- D2 pad 2: Net-(D1-A) -> /EN
Routing:
- net /EN: track 27.5 -> 70.3 mm
- net /EMITER: track 0.00 -> 14.8 mm
- net /BOOT0: track 19.2 -> 32.0 mm, vias 2 -> 3
- net /NRST: track 29.1 -> 34.5 mm
- net /ESP32_E: track 50.9 -> 45.9 mm
- net /IO00: track 29.3 -> 34.3 mm
- net /STM32: track 0.00 -> 3.63 mm
- net /SDA: track 32.4 -> 36.0 mm
- net /SWCLK: track 22.6 -> 19.4 mm
- net /ESP32: track 0.00 -> 2.97 mm
- net /PULSE: track 53.7 -> 56.4 mm
- net /SCL: track 42.1 -> 39.8 mm
- net Net-(U2A-+): track 2.29 -> 3.81 mm
- net Net-(R9-Pad1): track 14.1 -> 15.3 mm
- net Net-(U2A--): track 14.8 -> 15.9 mm
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Other:
- board size 78.2 x 40.8 mm -> 80.5 x 40.8 mm
- board text added: "ESP32"
- board text added: "STM32"

Commit message: New version
Version 2 created
Other:
- board text added: "${Revision}"
- board text removed: "v${Revision}"
Changed lines of the file:
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@@
     )
   )
-  (property "Revision" "0.1")
+  (property "Revision" "V0.2")
   (net 0 "")
   (net 1 "/OSC1")
@@
     (effects (font (size 0.8 0.8) (thickness 0.1)) (justify right))
   )
-  (gr_text "v${Revision}" (at 136.3 51.7) (layer "F.SilkS")
+  (gr_text "${Revision}" (at 136.3 51.7) (layer "F.SilkS")
     (effects (font (size 1.5 1.5) (thickness 0.3) bold) (justify left bottom))
   )
